Commit message: update ROS

File: UR5_ws/src/common_sensors/urdf/sensors/kinect2.gazebo.xacro (robot description, xacro)
@@ -5,5 +5,5 @@
     <sensor type="depth" name="${name}_ir_sensor">
       <always_on>true</always_on>
-      <update_rate>1.0</update_rate>
+      <update_rate>20.0</update_rate>
       <camera>
         <horizontal_fov>${57.0*M_PI/180.0}</horizontal_fov>
@@ -21,5 +21,5 @@
         <baseline>0.2</baseline>
         <alwaysOn>true</alwaysOn>
-        <updateRate>1.0</updateRate>
+        <updateRate>10.0</updateRate>
         <cameraName>${camera_name}_ir</cameraName>
         <imageTopicName>/${camera_name}/ir/image_raw</imageTopicName>
@@ -49,5 +49,5 @@
     <sensor type="depth" name="${name}_rgb_sensor">
       <always_on>true</always_on>
-      <update_rate>1.0</update_rate>
+      <update_rate>20.0</update_rate>
       <camera>
         <horizontal_fov>${57.0*M_PI/180.0}</horizontal_fov>
@@ -64,5 +64,5 @@
       <plugin name="${link_name}_controller" filename="libgazebo_ros_openni_kinect.so">
         <alwaysOn>true</alwaysOn>
-        <updateRate>1.0</updateRate>
+        <updateRate>10.0</updateRate>
         <cameraName>${camera_name}_rgb</cameraName>
         <imageTopicName>/${camera_name}/rgb/image_raw</imageTopicName>

File: UR5_ws/src/common_sensors/urdf/sensors/kinect2.urdf.xacro (robot description, xacro)
@@ -23,5 +23,5 @@
         <origin xyz="-0.102 -0.148 0" rpy="0 0 0"/>
         <geometry>
-          <mesh filename="package://common_sensors/meshes/sensors/kinect2_assembly.STL" scale="0.001 0.001 0.001" />
+          <mesh filename="package://common_sensors/meshes/sensors/kinect2_assembly.dae" scale="0.001 0.001 0.001" />
         </geometry>
         <material name="gray">
